File: pcb/pd.kicad_sch (KiCad schematic)
At the start: 0 parts

Commit message: feat: BME280 sensor
Other:
- note added: "TODO: - Solar Charger - USB Charger (fallback) - Buck-boost converter (MP28164)"
Changed lines of the file:
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@@
 	(generator_version "9.0")
 	(paper "A4")
+	(text "TODO:\n- Solar Charger\n- USB Charger (fallback)\n- Buck-boost converter (MP28164)"
+		(exclude_from_sim no)
+		(at 17.526 20.828 0)
+		(effects
+			(font
+				(size 1.27 1.27)
+			)
+			(justify left)
+		)
+	)
 )

Commit message: chore: docs
Other:
- company: (none) -> Ivan Leonard O Aparte <ivanleonard.aparte@cit.edu>
- title: (none) -> Banshee Power Schematics
Changed lines of the file:
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@@
 	(generator_version "9.0")
 	(paper "A4")
+	(title_block
+		(title "Banshee Power Schematics")
+		(date "2026-01-29")
+		(rev "1")
+		(company "Ivan Leonard O Aparte <ivanleonard.aparte@cit.edu>")
+		(comment 1 "TODO")
+	)
 	(text "TODO:\n- Solar Charger\n- USB Charger (fallback)\n- Buck-boost converter (MP28164)"
 		(exclude_from_sim no)

Commit message: chore: date update
Other:
- title: Banshee Power Schematics -> Banshee Microcontroller + Supporting Systems
Changed lines of the file:
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@@
 	(paper "A4")
 	(title_block
-		(title "Banshee Power Schematics")
-		(date "2026-01-29")
+		(title "Banshee Microcontroller + Supporting Systems")
+		(date "2026-02-05")
 		(rev "1")
 		(company "Ivan Leonard O Aparte <ivanleonard.aparte@cit.edu>")

Commit message: chore: :(
Other:
- note removed: "TODO: - Solar Charger - USB Charger (fallback) - Buck-boost converter (MP28164)"
Changed lines of the file:
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@@
 		(comment 1 "TODO")
 	)
-	(text "TODO:\n- Solar Charger\n- USB Charger (fallback)\n- Buck-boost converter (MP28164)"
-		(exclude_from_sim no)
-		(at 17.526 20.828 0)
-		(effects
-			(font
-				(size 1.27 1.27)
-			)
-			(justify left)
-		)
-	)
 )

Commit message: chore: page documentation
Other:
- title: Banshee Microcontroller + Supporting Systems -> Banshee Power Delivery System
Changed lines of the file:
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@@
 	(paper "A4")
 	(title_block
-		(title "Banshee Microcontroller + Supporting Systems")
-		(date "2026-02-05")
+		(title "Banshee Power Delivery System")
+		(date "2026-02-18")
 		(rev "1")
 		(company "Ivan Leonard O Aparte <ivanleonard.aparte@cit.edu>")
-		(comment 1 "TODO")
+		(comment 1 "STEM 12 - Altruism | S.Y. 2025-2026")
 	)
 )

Commit message: feat: 3.3V power supply
Parts:
- added C23, C25, C26: 10u, symbol Device:C
- added C24: 1n, symbol Device:C
- added L1: 1.5u, symbol Device:L
- added R16: 1M R, symbol Device:R
- added U8: TPS63051RMWR, Banshee:QFN50P250X250X100-12N, symbol Banshee:TPS63051RMWR
Connections:
- new net: L1.1, U8.1 (L1)
- new net: L1.2, U8.3 (L2)
- new net: C24.1, U8.7 (SS)
- new net: R16.2, U8.8 (PG)
- new net +3.3V: C25.1, C26.1, R16.1, U8.4 (VOUT), U8.5 (FB)
- new net GND: C23.2, C24.2, C25.2, C26.2, U8.2 (GND), U8.6 (PFM/PWM), U8.9 (GND)
- new net VCC: C23.1, U8.12 (VIN)
Other:
- note added: "3.3V @ 500mA Power Supply"

Commit message: chore: wiring of EN and ILIM0 pins
Connections:
- net VCC: now also U8.10 (ILIM0), U8.11 (EN)
Changed lines of the file:
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@@
 		(color 0 0 0 0)
 	)
+	(junction
+		(at 45.72 45.72)
+		(diameter 0)
+		(color 0 0 0 0)
+	)
+	(junction
+		(at 45.72 43.18)
+		(diameter 0)
+		(color 0 0 0 0)
+	)
 	(wire
 		(pts
@@
 	(wire
 		(pts
+			(xy 52.07 45.72) (xy 45.72 45.72)
+		)
+		(stroke
+			(width 0)
+			(type default)
+		)
+	)
+	(wire
+		(pts
 			(xy 52.07 55.88) (xy 46.99 55.88)
 		)
@@
 	(wire
 		(pts
+			(xy 45.72 43.18) (xy 52.07 43.18)
+		)
+		(stroke
+			(width 0)
+			(type default)
+		)
+	)
+	(wire
+		(pts
+			(xy 45.72 45.72) (xy 45.72 43.18)
+		)
+		(stroke
+			(width 0)
+			(type default)
+		)
+	)
+	(wire
+		(pts
 			(xy 67.31 67.31) (xy 67.31 63.5)
 		)
@@
 	(wire
 		(pts
+			(xy 45.72 48.26) (xy 45.72 45.72)
+		)
+		(stroke
+			(width 0)
+			(type default)
+		)
+	)
+	(wire
+		(pts
 			(xy 52.07 40.64) (xy 52.07 29.21)
 		)
@@
 	(wire
 		(pts
+			(xy 52.07 48.26) (xy 45.72 48.26)
+		)
+		(stroke
+			(width 0)
+			(type default)
+		)
+	)
+	(wire
+		(pts
 			(xy 31.75 46.99) (xy 31.75 43.18)
 		)
@@
 	(wire
 		(pts
-			(xy 31.75 43.18) (xy 52.07 43.18)
-		)
-		(stroke
+			(xy 31.75 43.18) (xy 45.72 43.18)
+		)
+		(stroke

Commit message: fix: reset wiring
Parts:
- R16: value 1M R -> 47k
- U8: JLCPCB Part# (none) -> C139412
Connections:
- net MCU ~{RESET}: now reaches R16.2, U8.8 (PG)
Changed lines of the file:
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@@
+	)
+	(junction
+		(at 87.63 55.88)
+		(diameter 0)
+		(color 0 0 0 0)
 	)
 	(junction
@@
 	(wire
 		(pts
+			(xy 87.63 55.88) (xy 90.17 55.88)
+		)
+		(stroke
+			(width 0)
+			(type default)
+		)
+	)
+	(wire
+		(pts
 			(xy 66.04 69.85) (xy 66.04 67.31)
 		)
@@
 			(width 0)
 			(type default)
+		)
+	)
+	(hierarchical_label "MCU ~{RESET}"
+		(shape output)
+		(at 90.17 55.88 0)
+		(effects
+			(font
+				(size 1.27 1.27)
+			)
+			(justify left)
 		)
 	)
@@
 			)
 		)
+		(property "JLCPCB Part#" "C139412"
+			(at 66.04 49.53 0)
+			(effects
+				(font
+					(size 1.27 1.27)
+				)
+				(hide yes)
+			)
+		)
 		(pin "4"
 		)
@@
 			)
 		)
-		(property "Value" "1M R"
+		(property "Value" "47k"
 			(at 90.17 50.7999 0)
 			(effects
